File: pcb/PNCATEHO_v3/PNCATEHO_v3.kicad_sch (KiCad schematic)
At the start: 27 parts, among them J1 TestPoint_2Pole, SW1 SW_PUSH, SW10 SW_PUSH, SW2 SW_PUSH, SW3 SW_PUSH, SW4 SW_PUSH, SW5 SW_PUSH, SW6 SW_PUSH, SW7 SW_PUSH, SW8 SW_PUSH, SW9 SW_PUSH, U1 ProMicro_r

Commit message: fix title
Other:
- note added: "А"
- note added: "Е"
- note added: "И"
- note added: "Н"
- note added: "О"
- note added: "Р"
- note added: "С"
- note added: "Т"
