File: pcb/PNCATEHO_v4/PNCATEHO_v4.kicad_sch (KiCad schematic)
At the start: 27 parts, among them J1 TestPoint_2Pole, SW1 SW_PUSH, SW10 SW_PUSH, SW2 SW_PUSH, SW3 SW_PUSH, SW4 SW_PUSH, SW5 SW_PUSH, SW6 SW_PUSH, SW7 SW_PUSH, SW8 SW_PUSH, SW9 SW_PUSH, U1 ProMicro_r

Commit message: Library change, change to hs switches, led changes
Parts:
- H1, H2, H3: footprint enki_lib:HOLE -> PNCATEHO:Hole
- J1: footprint enki_lib:battery_conn -> PNCATEHO:battery_conn_duplex
- PSW1: footprint enki_lib:switch_MSK-12C02_smd -> PNCATEHO:MSK-12C02_DUAL
- SW1, SW10, SW2, SW3, SW4, SW5, SW6, SW7, SW8, SW9: footprint keyswitches-pretty:Kailh_socket_PG1350_reversible -> PNCATEHO:Kailh_socket_PG1350_reversible
Changed lines of the file:
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@@
 			)
 		)
-		(property "Footprint" "keyswitches-pretty:Kailh_socket_PG1350_reversible"
+		(property "Footprint" "PNCATEHO:Kailh_socket_PG1350_reversible"
 			(at 80.01 21.082 0)
 			(effects
@@
 			)
 		)
-		(property "Footprint" "keyswitches-pretty:Kailh_socket_PG1350_reversible"
+		(property "Footprint" "PNCATEHO:Kailh_socket_PG1350_reversible"
 			(at 97.79 21.082 0)
 			(effects
@@
 			)
 		)
-		(property "Footprint" "keyswitches-pretty:Kailh_socket_PG1350_reversible"
+		(property "Footprint" "PNCATEHO:Kailh_socket_PG1350_reversible"
 			(at 115.57 21.082 0)
 			(effects
@@
 			)
 		)
-		(property "Footprint" "keyswitches-pretty:Kailh_socket_PG1350_reversible"
+		(property "Footprint" "PNCATEHO:Kailh_socket_PG1350_reversible"
 			(at 133.35 21.082 0)
 			(effects
@@
 			)
 		)
-		(property "Footprint" "keyswitches-pretty:Kailh_socket_PG1350_reversible"
+		(property "Footprint" "PNCATEHO:Kailh_socket_PG1350_reversible"
 			(at 80.01 36.322 0)
 			(effects
@@
 			)
 		)
-		(property "Footprint" "keyswitches-pretty:Kailh_socket_PG1350_reversible"
+		(property "Footprint" "PNCATEHO:Kailh_socket_PG1350_reversible"
 			(at 97.79 36.322 0)
 			(effects
@@
 			)
 		)
-		(property "Footprint" "keyswitches-pretty:Kailh_socket_PG1350_reversible"
+		(property "Footprint" "PNCATEHO:Kailh_socket_PG1350_reversible"
 			(at 115.57 36.322 0)
 			(effects
@@
 			)
 		)
-		(property "Footprint" "keyswitches-pretty:Kailh_socket_PG1350_reversible"
+		(property "Footprint" "PNCATEHO:Kailh_socket_PG1350_reversible"
 			(at 133.35 36.322 0)
 			(effects
@@
 			)
 		)
-		(property "Footprint" "keyswitches-pretty:Kailh_socket_PG1350_reversible"
+		(property "Footprint" "PNCATEHO:Kailh_socket_PG1350_reversible"
 			(at 133.35 51.562 0)
 			(effects
@@
 			)
 		)
-		(property "Footprint" "keyswitches-pretty:Kailh_socket_PG1350_reversible"
+		(property "Footprint" "PNCATEHO:Kailh_socket_PG1350_reversible"
 			(at 151.13 51.562 0)
 			(effects
@@
 			)
 		)
-		(property "Footprint" "enki_lib:HOLE"
+		(property "Footprint" "PNCATEHO:Hole"
 			(at 88.138 26.924 0)
 			(effects
@@
 			)
 		)
-		(property "Footprint" "enki_lib:battery_conn"
+		(property "Footprint" "PNCATEHO:battery_conn_duplex"
 			(at 15.621 28.194 0)
 			(effects
@@
 			)
 		)
-		(property "Footprint" "enki_lib:HOLE"
+		(property "Footprint" "PNCATEHO:Hole"
 			(at 148.59 42.672 0)
 			(effects
@@
 			)
 		)
-		(property "Footprint" "enki_lib:HOLE"
+		(property "Footprint" "PNCATEHO:Hole"
 			(at 126.492 26.924 0)
 			(effects
@@
 			)
 		)
-		(property "Footprint" "enki_lib:switch_MSK-12C02_smd"
+		(property "Footprint" "PNCATEHO:MSK-12C02_DUAL"
 			(at 20.701 23.114 0)
 			(effects
