File: pcb/PNCATEHO_v5/PNCATEHO_v5.kicad_sch (KiCad schematic)
At the start: 27 parts, among them J1 TestPoint_2Pole, SW1 SW_PUSH, SW10 SW_PUSH, SW2 SW_PUSH, SW3 SW_PUSH, SW4 SW_PUSH, SW5 SW_PUSH, SW6 SW_PUSH, SW7 SW_PUSH, SW8 SW_PUSH, SW9 SW_PUSH, U1 ProMicro_r

Commit message: Basic layout
Connections:
- no-connect marks 8 -> 9
Changed lines of the file:
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@@
+	)
+	(no_connect
+		(at 25.781 25.654)
 	)
 	(no_connect

Commit message: v0.5.1 100x100 version pcb
Parts:
- U1: footprint PNCATEHO:ProMicro_duplex -> PNCATEHO:ProMicro_duplex_mirrored
Changed lines of the file:
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@@
 			)
 		)
-		(property "Footprint" "PNCATEHO:ProMicro_duplex"
+		(property "Footprint" "PNCATEHO:ProMicro_duplex_mirrored"
 			(at 41.148 26.1366 0)
 			(effects
