File: pcb/PNCATEHO_MK_DOSE/PNCATEHO_MK_DOSE.kicad_sch (KiCad schematic)
At the start: 47 parts, among them J1 TestPoint_2Pole, U1 ProMicro_r

Commit message: PNCATEHO MK-DOSE routed
Parts:
- removed LED1, LED10, LED2, LED3, LED4, LED5, LED6, LED7, LED8, LED9: YS-SK6812MINI-E, PNCATEHO:YS-SK6812MINI-E_duplex, symbol PNCATEHO:YS-SK6812MINI-E
- removed PSW1: SW_SPDT, PNCATEHO:MSK-12C02_DUAL, symbol Switch:SW_SPDT
- added D21, D22, D23: LED, PNCATEHO:0603-led_dual, symbol Device:LED
- added PSW1: ~, PNCATEHO:bsi10h, symbol PNCATEHO:bsi10h
- added R1, R2, R3: R, PNCATEHO:0603-resistor_dual, symbol Device:R
- D1, D10, D11, D12, D13, D14, D15, D16, D17, D18, D19, D2, D20, D3, D4, D5, D6, D7, D8, D9: footprint Diode_SMD:D_SOD-123 -> PNCATEHO:D3_SMD
Connections:
- net LED is gone; now on net R5: U1.12 (B5/9)
- net C0: now also U1.19 (A2/F5); no longer U1.20 (A3/F4)
- net C1: now also U1.10 (E6/7); no longer U1.19 (A2/F5)
- net C2: now also U1.17 (A0/F7); no longer U1.18 (A1/F6)
- net C3: now also U1.16 (15/B1); no longer U1.17 (A0/F7)
- net GND: now also D21.1 (K), D22.1 (K), D23.1 (K)
- net R0: now also U1.20 (A3/F4); no longer U1.10 (E6/7)
- net R1: now also U1.18 (A1/F6); no longer U1.11 (B4/8)
- net R2: now also U1.15 (14/B3); no longer U1.16 (15/B1)
- net R3: now also U1.11 (B4/8); no longer U1.15 (14/B3)
- net R4: now also U1.13 (10/B6); no longer U1.14 (16/B2)
- net R5: no longer U1.13 (10/B6)
- net VBAT: now also PSW1.2
- net VCC: no longer U1.21 (VCC)
- net LED0: now reaches U1.7 (D4/4)
- net LED0: now also R1.2
- net LED1: now reaches U1.8 (C6/5)
- net LED1: now also R2.2
- net LED2: now reaches U1.9 (D7/6)
- net LED2: now also R3.2
- net at J1.1: now also PSW1.1
- new net: D23.2 (A), R3.1
- new net: D21.2 (A), R1.1
- new net: D22.2 (A), R2.1
- no-connect marks 9 -> 7
Other:
- moved on the sheet: RSW1

Commit message: MK-DOSE version, with 100x100 version
Parts:
- U1: footprint PNCATEHO:ProMicro_duplex -> PNCATEHO:ProMicro_duplex_mirrored
Changed lines of the file:
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@@
 			)
 		)
-		(property "Footprint" "PNCATEHO:ProMicro_duplex"
+		(property "Footprint" "PNCATEHO:ProMicro_duplex_mirrored"
 			(at 41.91 25.8826 0)
 			(effects
